File: Main_Board/PowerRelay.kicad_pcb (KiCad board)
At the start: 2 copper layers, 100 x 100 mm, 29 parts, among them J1 Screw_Terminal_01x03, J2 Conn_01x20_Female, J3 Conn_01x20_Female, J5 Screw_Terminal_01x03, J6 Screw_Terminal_01x03, J8 AudioJack4, K1 G5LE-1A4_DC3, K2 G5LE-1A4_DC3, Q1 2N7000, Q2 2N7000

Commit message: multiple changes and convert to ki cad 7
Parts:
- removed the H5 at (109.0, 61.0)
- added F3: Fuse, 39105000000:39105000000, F.Cu at (110.9, 51.8)
- added J4: Conn_01x02_Female, Connector_PinHeader_2.54mm:PinHeader_1x02_P2.54mm_Vertical, F.Cu at (110.0, 63.0)
- moved H5 2.24 mm to (90.0, 59.0)
- moved A1 1.28 mm to (100.1, 92.9)
- moved J2 1.28 mm to (84.1, 117.0)
- moved J3 1.28 mm to (116.0, 68.7)
- moved G*** 0.89 mm to (117.0, 129.0)
- renumbered H6 to H5
Connections:
- J8 pad 1: (no net) -> GND
- J8 pad 2: (no net) -> RX
- J8 pad 3: (no net) -> TX
- J8 pad 4: (no net) -> Net-(F3-Pad1)
Routing:
- net +3V3: track 216.3 -> 202.8 mm
- net Net-(F3-Pad1): track 0.00 -> 12.1 mm
- net Net-(J4-Pin_1): track 0.00 -> 4.82 mm
- net Heating: track 18.4 -> 21.0 mm
- net Cooling: track 12.1 -> 13.8 mm
- net Earth: track 236.7 -> 238.3 mm
- net RX: track 22.4 -> 23.8 mm
- net TX: track 15.5 -> 16.8 mm
- net VAC: track 157.0 -> 155.9 mm
- net Net-(PS1-AC(N)): track 57.9 -> 59.0 mm
- net Net-(F1-Pad2): track 22.7 -> 21.7 mm
- net Net-(J5-Pin_2): track 23.1 -> 23.6 mm
- net Net-(J6-Pin_2): track 22.3 -> 22.8 mm
Other:
- outline, holes or cut-outs redrawn
